File: PCB/hackpad.kicad_pcb (KiCad board)
At the start: 2 copper layers, 58.8 x 53.3 mm, 8 parts, among them M1 Module_XIAO-RP2040, SW1 SW_Push, SW2 SW_Push, SW3 SW_Push, SW4 RotaryEncoder_Switch, SW5 RotaryEncoder_Switch, SW6 SW_Push, SW7 SW_Push

Commit message: read me initial
Routing:
- added copper zone on F.Cu, net GND
Other:
- board text added: "heian my569 myMacropad v1 2026"
- board text removed: "heian my569 macropad v1 2026"
Changed lines of the file:
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@@
 			(outputformat 1)
 			(mirror no)
-			(drillshape 0)
+			(drillshape 1)
 			(scaleselection 1)
-			(outputdirectory "../../Downloads/Projects/Hackpad/PCB & Schematic/")
+			(outputdirectory "")
 		)
 	)
@@
 		(layer "Edge.Cuts")
 	)
-	(gr_text "heian\nmy569\nmacropad v1\n2026\n"
+	(gr_text "heian\nmy569\nmyMacropad v1\n2026\n"
 		(at 91.7 123.1 0)
 		(layer "F.SilkS")
@@
 		(start 135 100.1)
 		(end 147 100.1)
-		(width 0.2)
+		(width 1)
 		(layer "F.Cu")
 		(net "GND")
@@
 		(net "/B4")
 	)
+	(zone
+		(net "GND")
+		(layer "F.Cu")
+		(hatch edge 0.5)
+		(connect_pads
+			(clearance 0.5)
+		)
+		(min_thickness 0.25)
+		(fill yes
+			(thermal_gap 0.5)
+			(thermal_bridge_width 0.5)
+			(island_removal_mode 0)
+		)
+		(polygon
+			(pts
+				(xy 94.4 92.42) (xy 93.9 141.8) (xy 138.5 139.4) (xy 136.4 96.5)
+			)
+		)
+	)
 	(embedded_fonts no)
